File: Hardware/C8W1B1V1.0/Kicad/C8W1B1V1.0.kicad_pcb (KiCad board)
At the start: 4 copper layers, 22 x 46 mm, 43 parts, among them IC1 AT25DF021A-MAHN-T, IC2 S2-LPQTR, IC3 BALF-SPI2-01D3, IC4 MB85RS64TPN-G-AMEWE1, J1 Conn_01x07, J2 Conn_01x07_Pin, U1 STM32G081KBUx, Y1 NX1612SA-50M-EXS00A-CS08403

Commit message: Dodano nazwę na PCB
Other:
- board text added: "C8W1B1V1.0"
Changed lines of the file:
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@@
+		)
+	)
+	(gr_text "C8W1B1V1.0"
+		(at 138.78 108.99 90)
+		(layer "F.SilkS")
+		(effects
+			(font
+				(size 1 1)
+				(thickness 0.1)
+			)
+			(justify left bottom)
 		)
 	)
