File: Hardware/C8W1B1V1.0/Kicad/Radio.kicad_sch (KiCad schematic)
At the start: 25 parts, among them IC2 S2-LPQTR, IC3 BALF-SPI2-01D3, Y1 NX1612SA-50M-EXS00A-CS08403

Commit message: Dodano nazwę na PCB
Parts:
- L1: value LQG15HS12NJD2D -> LQG15HS12NH02D
Changed lines of the file:
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@@
 			)
 		)
-		(property "Value" "LQG15HS12NJD2D"
+		(property "Value" "LQG15HS12NH02D"
 			(at 217.17 193.04 90)
 			(effects
